Commit message: updating yaml

File: urdf/gem_e2.urdf (robot description, URDF)
Before this commit: robot GEM, 18 links, 17 joints
Joints:
- joint base-imu: origin xyz=0.770 0 0.320 rpy=0 0 0 -> xyz=0.770 0 0.320 rpy=0 0 -1.571
- joint rack-gps: origin xyz=-0.35 -0.624 0.025 rpy=0 0 0 -> xyz=-0.35 -0.624 0.025 rpy=0 0 -1.571
